Commit message: Visualize the sensors by default in Gazebo

File: mirte_description/mirte_master_description/urdf/lidar.xacro (robot description, xacro)
@@ -72,49 +72,8 @@
     <xacro:property name="lidar_sensor_link" value="lidar_link" />
   </xacro:unless>
-<!--
-  <gazebo reference="lidar_link">
-    <sensor type="ray" name="lidar">
-      <xacro:if value="$(arg use_correct_laser_frame)">
-        <pose>0 0 0 0 0 0</pose>
-      </xacro:if>
-      <xacro:unless value="$(arg use_correct_laser_frame)">
-        <pose>0 0 0 0 0 0</pose>
-      </xacro:unless>
-      <visualize>false</visualize>
-      <update_rate>10</update_rate>
-      <ray>
-        <scan>
-          <horizontal>
-            <samples>500</samples>
-            <resolution>1</resolution>
-            <min_angle>${-pi}</min_angle>
-            <max_angle>${pi}</max_angle>
-          </horizontal>
-        </scan>
-        <range>
-          <min>0.05</min>
-          <max>10.0</max>
-          <resolution>0.015</resolution>
-        </range>
-        <noise>
-          <type>gaussian</type>
-          <mean>0.0</mean>
-          <stddev>0.01</stddev>
-        </noise>
-      </ray>
-      <plugin name="gazebo_lidar" filename="libgazebo_ros_laser.so">
-        <ros>
-          <remapping>~/out:=scan</remapping>
-        </ros>
-        <output_type>sensor_msgs/LaserScan</output_type>
-        <frame_name>${lidar_sensor_link}</frame_name>
-      </plugin>
-    </sensor>
-  </gazebo>
--->
   <gazebo reference="lidar_link">
         <sensor name="lidar" type="ray">
             <pose> 0 0 0 0 0 0 </pose>
-            <visualize>false</visualize>
+            <visualize>${visualize_sensors}</visualize>
             <update_rate>10</update_rate>
             <ray>

File: mirte_description/mirte_master_description/urdf/mirte_master.xacro (robot description, xacro)
@@ -20,4 +20,5 @@
   <xacro:property name="wheel_effort" value="5" />
   <xacro:property name="base_mass" value="5.0" />
+  <xacro:property name="visualize_sensors" value="True" />
   <material name="blue">
     <color rgba="0.203125 0.23828125 0.28515625 1.0" />

File: mirte_description/mirte_master_description/urdf/ultrasonic.xacro (robot description, xacro)
@@ -22,5 +22,5 @@
     <gazebo reference="base_sonar_${name}">
       <sensor type="ray" name="range_sensor_${name}">
-        <visualize>false</visualize>
+        <visualize>${visualize_sensors}</visualize>
           <ray>
             <scan>
