Commit message: Cleanup of mecanum wheels xacro

File: mirte_description/mirte_master_description/urdf/mirte_master.xacro (robot description, xacro)
@@ -3,23 +3,14 @@
   name="mirte_master" xmlns:xacro="http://ros.org/wiki/xacro">
   <xacro:arg name="flag_enable" default="False" />
-  <xacro:arg name="arm_enable" default="False" />
+  <xacro:arg name="arm_enable" default="True" />
   <xacro:arg name="screen_enable" default="False" />
   <xacro:arg name="front_camera_enable" default="False" />
-  <xacro:arg name="sonar_enable" default="False" />
-  <xacro:arg name="lidar_enable" default="False" />
+  <xacro:arg name="sonar_enable" default="True" />
+  <xacro:arg name="lidar_enable" default="True" />
   <xacro:arg name="depth_camera_enable" default="True" />
-  <xacro:arg name="imu_enable" default="False" />
-  <xacro:arg name="use_namespace" default="False"/>
-  <xacro:arg name="namespace_name" default="" />
-  <xacro:if value="$(arg use_namespace)" >
-    <xacro:property name="camera_name" value="$(arg namespace_name)/camera" lazy_eval="False"/>
-    <xacro:property name="namespace" value="$(arg namespace_name)" scope="global" lazy_eval="False"/>
-    <xacro:property name="tf_namespace" value="$(arg namespace_name)/" scope="global" lazy_eval="False"/>
-  </xacro:if>
-  <xacro:unless value="$(arg use_namespace)">
-    <xacro:property name="camera_name" value="camera" lazy_eval="False"/>
-    <xacro:property name="namespace" value="" scope="global" lazy_eval="False"/>
-    <xacro:property name="tf_namespace" value="" scope="global" lazy_eval="False"/>
-  </xacro:unless>
+  <xacro:arg name="imu_enable" default="True" />
+  <xacro:property name="camera_name" value="camera" lazy_eval="False"/>
+  <xacro:property name="namespace" value="" scope="global" lazy_eval="False"/>
+  <xacro:property name="tf_namespace" value="" scope="global" lazy_eval="False"/>
   <xacro:arg name="use_correct_laser_frame" default="True" />
   <xacro:property name="wheel_radius" value="0.050" />
@@ -98,188 +89,29 @@
     </collision>
   </link>
-  <link
-    name="wheel_left_front">
-    <inertial>
-      <origin xyz="0 0 0.025" />
-      <mass value="${wheel_mass}" />
-      <inertia
-        ixx="${wheel_mass * (3 * (wheel_radius**2) + (wheel_length**2)) / 12}"
-        iyy="${wheel_mass * (3 * (wheel_radius**2) + (wheel_length**2)) / 12}"
-        izz="${wheel_mass * (wheel_radius **2) / 2}"
-        ixy="0" ixz="0" iyz="0" />
-    </inertial>
-    <visual>
-      <geometry>
-        <mesh
-          filename="file://$(find mirte_master_description)/meshes/wheel_left_front.STL" />
-      </geometry>
-      <material name="">
-        <color rgba="0.79216 0.81961 0.93333 1" />
-      </material>
-    </visual>
-    <collision>
-      <origin xyz="0 0 0.025" />
-      <geometry>
-        <cylinder radius="${wheel_radius}" length="${wheel_length}" />
-      </geometry>
-    </collision>
-  </link>
-  <joint
-    name="wheel_left_front_joint"
-    type="continuous">
-    <origin
-      xyz="0.153 -0.085 -0.0455"
-      rpy="1.5708 0 -1.5708" />
-    <parent link="frame_link" />
-    <child link="wheel_left_front" />
-    <axis xyz="0 0 -1" />
-  </joint>
-  <transmission name="wheel_left_front_transmission">
-    <type>transmission_interface/SimpleTransmission</type>
-    <joint name="wheel_left_front_joint">
-      <hardwareInterface>hardware_interface/VelocityJointInterface</hardwareInterface>
-    </joint>
-    <actuator name="wheel_left_front_actuator">
-      <mechanicalReduction>1</mechanicalReduction>
-    </actuator>
-  </transmission>
-  <link
-    name="wheel_left_rear">
-    <inertial>
-      <origin xyz="0 0 0.025" />
-      <mass value="${wheel_mass}" />
-      <inertia
-        ixx="${wheel_mass * (3 * (wheel_radius**2) + (wheel_length**2)) / 12}"
-        iyy="${wheel_mass * (3 * (wheel_radius**2) + (wheel_length**2)) / 12}"
-        izz="${wheel_mass * (wheel_radius **2) / 2}"
-        ixy="0" ixz="0" iyz="0" />
-    </inertial>
-    <visual>
-      <geometry>
-        <mesh
-          filename="file://$(find mirte_master_description)/meshes/wheel_left_rear.STL" />
-      </geometry>
-      <material name="">
-        <color rgba="0.79216 0.81961 0.93333 1" />
-      </material>
-    </visual>
-    <collision>
-      <origin xyz="0 0 0.025" />
-      <geometry>
-        <cylinder radius="${wheel_radius}" length="${wheel_length}" />
-      </geometry>
-    </collision>
-  </link>
-  <joint
-    name="wheel_left_rear_joint"
-    type="continuous">
-    <origin
-      xyz="0.153 0.085 -0.0455"
-      rpy="1.5708 0 -1.5708" />
-    <parent link="frame_link" />
-    <child link="wheel_left_rear" />
-    <axis xyz="0 0 -1" />
-  </joint>
-  <transmission name="wheel_left_rear_transmission">
-    <type>transmission_interface/SimpleTransmission</type>
-    <joint name="wheel_left_rear_joint">
-      <hardwareInterface>hardware_interface/VelocityJointInterface</hardwareInterface>
-    </joint>
-    <actuator name="wheel_left_rear_actuator">
-      <mechanicalReduction>1</mechanicalReduction>
-    </actuator>
-  </transmission>
-  <link
-    name="wheel_right_front">
-    <inertial>
-      <origin xyz="0 0 -0.025" />
-      <mass value="${wheel_mass}" />
-      <inertia
-        ixx="${wheel_mass * (3 * (wheel_radius**2) + (wheel_length**2)) / 12}"
-        iyy="${wheel_mass * (3 * (wheel_radius**2) + (wheel_length**2)) / 12}"
-        izz="${wheel_mass * (wheel_radius **2) / 2}"
-        ixy="0" ixz="0" iyz="0" />
-    </inertial>
-    <visual>
-      <geometry>
-        <mesh
-          filename="file://$(find mirte_master_description)/meshes/wheel_right_front.STL" />
-      </geometry>
-      <material name="">
-        <color rgba="0.79216 0.81961 0.93333 1" />
-      </material>
-    </visual>
-    <collision>
-      <origin xyz="0 0 -0.025" />
-      <geometry>
-        <cylinder radius="${wheel_radius}" length="${wheel_length}" />
-      </geometry>
-    </collision>
-  </link>
-  <joint
-    name="wheel_right_front_joint"
-    type="continuous">
-    <origin
-      xyz="-0.153 -0.085 -0.0455"
-      rpy="1.5708 0 -1.5708" />
-    <parent link="frame_link" />
-    <child link="wheel_right_front" />
-    <axis xyz="0 0 -1" />
-  </joint>
-  <transmission name="wheel_right_front_transmission">
-    <type>transmission_interface/SimpleTransmission</type>
-    <joint name="wheel_right_front_joint">
-      <hardwareInterface>hardware_interface/VelocityJointInterface</hardwareInterface>
-    </joint>
-    <actuator name="wheel_right_front_actuator">
-      <mechanicalReduction>1</mechanicalReduction>
-    </actuator>
-  </transmission>
-  <link
-    name="wheel_right_rear">
-    <inertial>
-      <origin xyz="0 0 -0.025" />
-      <mass value="${wheel_mass}" />
-      <inertia
-        ixx="${wheel_mass * (3 * (wheel_radius**2) + (wheel_length**2)) / 12}"
-        iyy="${wheel_mass * (3 * (wheel_radius**2) + (wheel_length**2)) / 12}"
-        izz="${wheel_mass * (wheel_radius **2) / 2}"
-        ixy="0" ixz="0" iyz="0" />
-    </inertial>
-    <visual>
-      <geometry>
-        <mesh
-          filename="file://$(find mirte_master_description)/meshes/wheel_right_rear.STL" />
-      </geometry>
-      <material name="">
-        <color rgba="0.79216 0.81961 0.93333 1" />
-      </material>
-    </visual>
-    <collision>
-      <origin xyz="0 0 -0.025" />
-      <geometry>
-        <cylinder radius="${wheel_radius}" length="${wheel_length}" />
-      </geometry>
-    </collision>
-  </link>
-  <joint
-    name="wheel_right_rear_joint"
-    type="continuous">
-    <origin
-      xyz="-0.153 0.085 -0.0455"
-      rpy="1.5708 0 -1.5708" />
-    <parent link="frame_link" />
-    <child link="wheel_right_rear" />
-    <axis xyz="0 0 -1" />
-  </joint>
-  <transmission name="wheel_right_rear_transmission">
-    <type>transmission_interface/SimpleTransmission</type>
-    <joint name="wheel_right_rear_joint">
-      <hardwareInterface>hardware_interface/VelocityJointInterface</hardwareInterface>
-    </joint>
-    <actuator name="wheel_right_rear_actuator">
-      <mechanicalReduction>1</mechanicalReduction>
-    </actuator>
-  </transmission>
+  <xacro:include filename="$(find mirte_master_description)/urdf/wheel.xacro" />
+   <!-- 0.025   -1 -->
+    <xacro:mecanum_wheel name="left_front" wheel_type="left" link_origin="0.025">
+      <origin
+        xyz="${0.153 - 0} -0.085 -0.0455"
+        rpy="1.5708 0 -1.5708" />
+    </xacro:mecanum_wheel>
+   <!-- 0.025   -1 -->
+    <xacro:mecanum_wheel name="left_rear" wheel_type="right" link_origin="0.025">
+      <origin
+        xyz="${0.153 - 0} 0.085 -0.0455"
+        rpy="1.5708 0 -1.5708" />
+    </xacro:mecanum_wheel>
+   <!-- -0.025   -1 -->
+    <xacro:mecanum_wheel name="right_front" wheel_type="right" link_origin="-0.025">
+      <origin
+        xyz="${-0.153 + wheel_length} -0.085 -0.0455"
+        rpy="1.5708 0 -1.5708" />
+    </xacro:mecanum_wheel>
+   <!-- -0.025   -1 -->
+    <xacro:mecanum_wheel name="right_rear" wheel_type="left" link_origin="-0.025">
+      <origin
+        xyz="${-0.153 + wheel_length} 0.085 -0.0455"
+        rpy="1.5708 0 -1.5708" />
+    </xacro:mecanum_wheel>
   <xacro:if value="$(arg front_camera_enable)">
     <link

Commit message: add base_footprint to urdf

File: mirte_description/mirte_master_description/urdf/mirte_master.xacro (robot description, xacro)
@@ -161,4 +161,11 @@
     </joint>
   </xacro:if>
+  <xacro:property name="wheel_zoff" value="0.05"/>
+  <link name="base_footprint"/>
+  <joint name="base_joint" type="fixed">
+    <parent link="base_link"/>
+    <child link="base_footprint"/>
+    <origin xyz="0.0 0.0 ${-(wheel_radius + wheel_zoff)}" rpy="0 0 0"/>
+  </joint>
   <xacro:if value="$(arg sonar_enable)">
     <xacro:include filename="$(find mirte_master_description)/urdf/ultrasonic.xacro" />
